Commit message: On branch luna  Changes to be committed: 	new file:   bringup/config/imu.yaml 	modified:   bringup/config/localization.yaml 	modified:   bringup/launch/diffbot.launch.py 	modified:   description/urdf/diffbot_description.urdf.xacro 	modified:   launch/rplidar.launch.py 	modified:   package.xml

File: description/urdf/diffbot_description.urdf.xacro (robot description, xacro)
@@ -338,5 +338,5 @@
     </gazebo>
     <!-- FRONT LEFT WHEEL LINK -->
-    <joint name="left_wheel_joint" type="continuous">
+    <joint name="right_wheel_joint" type="continuous">
         <parent link="base_link"/>
         <child link="left_wheel"/>
@@ -364,5 +364,5 @@
     </gazebo>
     <!-- FRONT RIGHT WHEEL LINK -->
-    <joint name="right_wheel_joint" type="continuous">
+    <joint name="left_wheel_joint" type="continuous">
         <parent link="base_link"/>
         <child link="right_wheel"/>

Commit message: *  Added laser odom to ekf
 *  Used the following package for laser odom: https://github.com/AlexKaravaev/ros2_laser_scan_matcher

 * Updated URDF

On branch nav2
 	Changes to be committed:
		modified:   bringup/config/diffbot_controllers.yaml
		modified:   bringup/config/localization.yaml
		modified:   bringup/launch/diffbot.launch.py
		new file:   description/rviz/nav2_slam_config.rviz
		modified:   description/urdf/diffbot_description.urdf.xacro
		modified:   launch/launch_sim.launch.py
		modified:   launch/rplidar.launch.py
		new file:   world/random.world

File: description/urdf/diffbot_description.urdf.xacro (robot description, xacro)
@@ -7,16 +7,23 @@
     <xacro:include filename="depth_camera.xacro"/>
     <xacro:property name="chassis_length" value="1.3501" />
-    <xacro:property name="chassis_to_base_link" value="0.73595" />
+    <xacro:property name="chassis_to_base_link" value="0.4954" />
     <xacro:property name="profile_height" value="0.0254" />
     <xacro:property name="profile_width" value="0.0254" />
-    <xacro:property name="tower_height" value="0.508" />
+    <xacro:property name="tower_height" value="0.388" />
     <xacro:property name="wheel_radius" value="0.1778" />
     <xacro:property name="wheel_thickness" value="0.07" />
-    <xacro:property name="wheel_mass" value="0.05" />
-    <xacro:property name="front_wheel_offset_x" value="0.3876" />
-    <xacro:property name="back_wheel_offset_x" value="0.437" />
+    <xacro:property name="wheel_mass" value="56" />
+    <xacro:property name="front_wheel_offset_x" value="0.14" />
+    <xacro:property name="back_wheel_offset_x" value="0.49" />
     <xacro:property name="wheel_offset_y" value="0.3182" />
     <xacro:property name="wheel_offset_z" value="0.1778" />
-    <xacro:property name="caster_wheel_mass" value="0.01"/>
+    <xacro:property name="caster_wheel_mass" value="56"/>
+    <xacro:property name="double_prof_mass" value="0.235398773"/>
+    <xacro:property name="single_prof_mass" value="0.147601476"/>
+    <xacro:property name="spoke_mass" value="1.6"/>
+    <xacro:property name="motorgearbox_mass" value="136"/>
+    <xacro:property name="scoop_mass" value="196"/>
+    <xacro:property name="tiltingact_mass" value="38"/>
+    <xacro:property name="liftingact_mass" value="44"/>
     <!-- BASE LINK -->
     <link name="base_link">
@@ -57,5 +64,5 @@
             </geometry>
         </collision>
-        <xacro:inertial_box mass="0.5" x="${-chassis_length}" y="0.0508" z="${profile_height}">
+        <xacro:inertial_box mass="${double_prof_mass*chassis_length*100}" x="${-chassis_length}" y="0.0508" z="${profile_height}">
             <origin xyz="${chassis_length/2} 0 0" rpy="0 0 0"/>
         </xacro:inertial_box>
@@ -85,5 +92,5 @@
             </geometry>
         </collision>
-        <xacro:inertial_box mass="0.5" x="${-chassis_length}" y="0.0508" z="${profile_height}">
+        <xacro:inertial_box mass="${double_prof_mass*chassis_length*100}" x="${-chassis_length}" y="0.0508" z="${profile_height}">
             <origin xyz="${chassis_length/2} 0 0" rpy="0 0 0"/>
         </xacro:inertial_box>
@@ -112,9 +119,36 @@
             </geometry>
         </collision>
-        <xacro:inertial_box mass="0.5" x="${profile_width}" y="0.4702" z="${profile_height}">
+        <xacro:inertial_box mass="${single_prof_mass*47.02}" x="${profile_width}" y="0.4702" z="${profile_height}">
             <origin xyz="0 0 0" rpy="0 0 0"/>
         </xacro:inertial_box>
     </link>
     <gazebo reference="tower_base">
+        <material>Gazebo/White</material>
+    </gazebo>
+    <!-- TOWER MIDDLE -->
+    <joint name="tower_middle_" type="fixed">
+        <parent link="base_link"/>
+        <child link="tower_middle"/>
+        <origin xyz="0 0 0.08"/>
+    </joint>
+    <link name="tower_middle">
+        <visual>
+            <origin xyz="0 0 0"/>
+            <geometry>
+                <box size="${profile_width} 0.4702 ${profile_height}"/>
+            </geometry>
+            <material name="white"/>
+        </visual>
+        <collision>
+            <origin xyz="0 0 0"/>
+            <geometry>
+                <box size="${profile_width} 0.4702 ${profile_height}"/>
+            </geometry>
+        </collision>
+        <xacro:inertial_box mass="${single_prof_mass*47.02}" x="${profile_width}" y="0.4702" z="${profile_height}">
+            <origin xyz="0 0 0" rpy="0 0 0"/>
+        </xacro:inertial_box>
+    </link>
+    <gazebo reference="tower_middle">
         <material>Gazebo/White</material>
     </gazebo>
@@ -140,5 +174,5 @@
             </geometry>
         </collision>
-        <xacro:inertial_box mass="0.5" x="${profile_width}" y="${profile_width}" z="${tower_height}">
+        <xacro:inertial_box mass="${single_prof_mass*tower_height*100}" x="${profile_width}" y="${profile_width}" z="${tower_height}">
             <origin xyz="0 0 ${tower_height/2}" rpy="0 0 0"/>
         </xacro:inertial_box>
@@ -168,5 +202,5 @@
             </geometry>
         </collision>
-        <xacro:inertial_box mass="0.5" x="${profile_width}" y="${profile_width}" z="${tower_height}">
+        <xacro:inertial_box mass="${single_prof_mass*tower_height*100}" x="${profile_width}" y="${profile_width}" z="${tower_height}">
             <origin xyz="0 0 ${tower_height/2}" rpy="0 0 0"/>
         </xacro:inertial_box>
@@ -196,5 +230,5 @@
             </geometry>
         </collision>
-        <xacro:inertial_box mass="0.5" x="${profile_width}" y="0.4702" z="${profile_height*2}">
+        <xacro:inertial_box mass="${double_prof_mass*0.4702*100}" x="${profile_width}" y="0.4702" z="${profile_height*2}">
             <origin xyz="0 0 0" rpy="0 0 0"/>
         </xacro:inertial_box>
@@ -221,5 +255,5 @@
             </geometry>
         </collision>
-        <xacro:inertial_box mass="0.5" x="0.4572" y="${profile_width}" z="${profile_height}">
+        <xacro:inertial_box mass="${single_prof_mass*0.4572*100}" x="0.4572" y="${profile_width}" z="${profile_height}">
             <origin xyz="0 0 0" rpy="0 0 0"/>
         </xacro:inertial_box>
@@ -249,5 +283,5 @@
             </geometry>
         </collision>
-        <xacro:inertial_box mass="0.5" x="0.4572" y="${profile_width}" z="${profile_height}">
+        <xacro:inertial_box mass="${single_prof_mass*0.4572*100}" x="0.4572" y="${profile_width}" z="${profile_height}">
             <origin xyz="0 0 0" rpy="0 0 0"/>
         </xacro:inertial_box>
@@ -260,5 +294,5 @@
         <parent link="base_link"/>
         <child link="motor_base_front"/>
-        <origin xyz="0.426 0 0"/>
+        <origin xyz="0.1 0 0"/>
     </joint>
     <link name="motor_base_front">
@@ -276,5 +310,5 @@
             </geometry>
         </collision>
-        <xacro:inertial_box mass="0.1" x="${profile_width}" y="0.4702" z="${profile_height}">
+        <xacro:inertial_box mass="${single_prof_mass*0.4702*100}" x="${profile_width}" y="0.4702" z="${profile_height}">
             <origin xyz="0 0 0" rpy="0 0 0"/>
         </xacro:inertial_box>
@@ -287,5 +321,5 @@
         <parent link="base_link"/>
         <child link="motor_base_back"/>
-        <origin xyz="0.35 0 0"/>
+        <origin xyz="0.175 0 0"/>
     </joint>
     <link name="motor_base_back">
@@ -303,9 +337,93 @@
             </geometry>
         </collision>
-        <xacro:inertial_box mass="0.1" x="${profile_width}" y="0.4702" z="${profile_height}">
+        <xacro:inertial_box mass="${single_prof_mass*0.4702*100}" x="${profile_width}" y="0.4702" z="${profile_height}">
             <origin xyz="0 0 0" rpy="0 0 0"/>
         </xacro:inertial_box>
     </link>
     <gazebo reference="motor_base_back">
+        <material>Gazebo/White</material>
+    </gazebo>
+     <!-- DOSER PROFILE LEFT -->
+     <joint name="doser_profile_left" type="fixed">
+        <parent link="base_link"/>
+        <child link="doser_profile_left"/>
+        <origin xyz="-0.2286 -0.0760254 0.1" rpy="0 ${pi/7.5} 0"/>
+        <axis xyz="1 0 0"/>
+    </joint>
+    <link name="doser_profile_left">
+        <visual>
+            <origin xyz="0 0 0"/>
+            <geometry>
+                <box size="0.490 ${profile_width} ${profile_height}"/>
+            </geometry>
+            <material name="white"/>
+        </visual>
+        <collision>
+            <origin xyz="0 0 0"/>
+            <geometry>
+                <box size="0.490 ${profile_width} ${profile_height}"/>
+            </geometry>
+        </collision>
+        <xacro:inertial_box mass="${single_prof_mass*0.490*100}" x="0.490" y="${profile_width}" z="${profile_height}">
+            <origin xyz="0 0 0" rpy="0 0 0"/>
+        </xacro:inertial_box>
+    </link>
+    <gazebo reference="doser_profile_left">
+        <material>Gazebo/White</material>
+    </gazebo>
+    <!-- DOSER PROFILE RIGHT -->
+    <joint name="doser_profile_right" type="fixed">
+        <parent link="base_link"/>
+        <child link="doser_profile_right"/>
+        <origin xyz="-0.2286 0.0760254 0.1" rpy="0 ${pi/7.5} 0"/>
+        <axis xyz="1 0 0"/>
+    </joint>
+    <link name="doser_profile_right">
+        <visual>
+            <origin xyz="0 0 0"/>
+            <geometry>
+                <box size="0.490 ${profile_width} ${profile_height}"/>
+            </geometry>
+            <material name="white"/>
+        </visual>
+        <collision>
+            <origin xyz="0 0 0"/>
+            <geometry>
+                <box size="0.490 ${profile_width} ${profile_height}"/>
+            </geometry>
+        </collision>
+        <xacro:inertial_box mass="${single_prof_mass*0.490*100}" x="0.490" y="${profile_width}" z="${profile_height}">
+            <origin xyz="0 0 0" rpy="0 0 0"/>
+        </xacro:inertial_box>
+    </link>
+    <gazebo reference="doser_profile_right">
+        <material>Gazebo/White</material>
+    </gazebo>
+    <!-- DOSER PROFILE CONNECTION TOP -->
+    <joint name="doser_profile_top" type="fixed">
+        <parent link="base_link"/>
+        <child link="doser_profile_top"/>
+        <origin xyz="-0.4596 0 0.20245" rpy="0 ${pi/7.5} 0"/>
+        <axis xyz="1 0 0"/>
+    </joint>
+    <link name="doser_profile_top">
+        <visual>
+            <origin xyz="0 0 0"/>
+            <geometry>
+                <box size="${profile_width} 0.3075 ${profile_height}"/>
+            </geometry>
+            <material name="white"/>
+        </visual>
+        <collision>
+            <origin xyz="0 0 0"/>
+            <geometry>
+                <box size="${profile_width} 0.3075 ${profile_height}"/>
+            </geometry>
+        </collision>
+        <xacro:inertial_box mass="${single_prof_mass*0.3075*100}" x="${profile_width}" y="0.3075" z="${profile_height}">
+            <origin xyz="0 0 0" rpy="0 0 0"/>
+        </xacro:inertial_box>
+    </link>
+    <gazebo reference="doser_profile_top">
         <material>Gazebo/White</material>
     </gazebo>
@@ -314,5 +432,5 @@
         <parent link="base_link"/>
         <child link="motor"/>
-        <origin xyz="0.3879 0 0"/>
+        <origin xyz="0.145 0 0"/>
     </joint>
     <link name="motor">
@@ -320,5 +438,5 @@
             <origin xyz="0 0 0.0375"/>
             <geometry>
-                <box size="0.2 0.5 0.075"/>
+                <box size="0.15 0.5 0.075"/>
             </geometry>
             <material name="orange"/>
@@ -327,8 +445,8 @@
             <origin xyz="0 0 0.0375"/>
             <geometry>
-                <box size="0.2 0.5 0.075"/>
-            </geometry>
-        </collision>
-        <xacro:inertial_box mass="0.01" x="0.2" y="0.5" z="0.075">
+                <box size="0.15 0.5 0.075"/>
+            </geometry>
+        </collision>
+        <xacro:inertial_box mass="${motorgearbox_mass}" x="0.15" y="0.5" z="0.075">
             <origin xyz="0 0 0.0375" rpy="0 0 0"/>
         </xacro:inertial_box>
@@ -408,5 +526,5 @@
     </gazebo>
     <!-- BACK LEFT WHEEL LINK -->
-    <joint name="back_left_wheel_joint" type="continuous">
+    <joint name="back_left_wheel_joint" type="fixed">
         <parent link="base_link"/>
         <child link="back_left_wheel"/>
@@ -441,5 +559,5 @@
     </gazebo>
     <!-- BACK RIGHT WHEEL LINK -->
-    <joint name="back_right_wheel_joint" type="continuous">
+    <joint name="back_right_wheel_joint" type="fixed">
         <parent link="base_link"/>
         <child link="back_right_wheel"/>
@@ -473,4 +591,174 @@
         <mu2 value="0.001"/>
     </gazebo>
+    <!-- DOZER -->
+    <joint name="Dozer_left" type="fixed">
+        <parent link="base_link"/>
+        <child link="doser_left"/>
+        <origin xyz="-0.597 -0.1587525 0.2" rpy="0 ${pi/5.81} 0"/>
+        <axis xyz="1 0 0"/>
+    </joint>
+    <link name="doser_left">
+        <visual>
+            <origin xyz="0 0 0"/>
+            <geometry>
+                <box size="0.4153 0.005 0.307"/>
+            </geometry>
+            <material name="white"/>
+        </visual>
+        <collision>
+            <origin xyz="0 0 0"/>
+            <geometry>
+                <box size="0.4153 0.005 0.307"/>
+            </geometry>
+        </collision>
+        <xacro:inertial_box mass="49" x="0.4153" y="0.005" z="0.307">
+            <origin xyz="0 0 0" rpy="0 0 0"/>
+        </xacro:inertial_box>
+    </link>
+    <gazebo reference="doser_left">
+        <material>Gazebo/White</material>
+    </gazebo>
+    <joint name="Dozer_right" type="fixed">
+        <parent link="base_link"/>
+        <child link="doser_right"/>
+        <origin xyz="-0.597 0.1587525 0.2" rpy="0 ${pi/5.81} 0"/>
+        <axis xyz="1 0 0"/>
+    </joint>
+    <link name="doser_right">
+        <visual>
+            <origin xyz="0 0 0"/>
+            <geometry>
+                <box size="0.4153 0.005 0.307"/>
+            </geometry>
+            <material name="white"/>
+        </visual>
+        <collision>
+            <origin xyz="0 0 0"/>
+            <geometry>
+                <box size="0.4153 0.005 0.307"/>
+            </geometry>
+        </collision>
+        <xacro:inertial_box mass="49" x="0.4153" y="0.005" z="0.307">
+            <origin xyz="0 0 0" rpy="0 0 0"/>
+        </xacro:inertial_box>
+    </link>
+    <gazebo reference="doser_right">
+        <material>Gazebo/White</material>
+    </gazebo>
+    <joint name="Dozer_back" type="fixed">
+        <parent link="base_link"/>
+        <child link="doser_back"/>
+        <origin xyz="-0.4205 0 0.095" rpy="0 ${pi/5.81} 0"/>
+        <axis xyz="1 0 0"/>
+    </joint>
+    <link name="doser_back">
+        <visual>
+            <origin xyz="0 0 0"/>
+            <geometry>
+                <box size="0.005 0.3225 0.312"/>
+            </geometry>
+            <material name="white"/>
+        </visual>
+        <collision>
+            <origin xyz="0 0 0"/>
+            <geometry>
+                <box size="0.005 0.3225 0.312"/>
+            </geometry>
+        </collision>
+        <xacro:inertial_box mass="49" x="0.005" y="0.3225" z="0.312">
+            <origin xyz="0 0 0" rpy="0 0 0"/>
+        </xacro:inertial_box>
+    </link>
+    <gazebo reference="doser_back">
+        <material>Gazebo/White</material>
+    </gazebo>
+    <joint name="Dozer_base" type="fixed">
+        <parent link="base_link"/>
+        <child link="doser_base"/>
+        <origin xyz="-0.675 0 0.066" rpy="0 ${pi/5.81} 0"/>
+        <axis xyz="1 0 0"/>
+    </joint>
+    <link name="doser_base">
+        <visual>
+            <origin xyz="0 0 0"/>
+            <geometry>
+                <box size="0.4153 0.3225 0.005"/>
+            </geometry>
+            <material name="white"/>
+        </visual>
+        <collision>
+            <origin xyz="0 0 0"/>
+            <geometry>
+                <box size="0.4153 0.3225 0.005"/>
+            </geometry>
+        </collision>
+        <xacro:inertial_box mass="49" x="0.4153" y="0.3225" z="0.005">
+            <origin xyz="0 0 0" rpy="0 0 0"/>
+        </xacro:inertial_box>
+    </link>
+    <gazebo reference="doser_base">
+        <material>Gazebo/White</material>
+    </gazebo>
+    <!-- LIFTING ACTUATOR LEFT -->
+    <xacro:property name="actuator_fixed_length" value="0.4575" />
+    <xacro:property name="actuator_extension_length" value="0.2" />
+    <xacro:property name="actuator_radius" value="0.02" />
+    <!-- FIXED PART -->
+    <joint name="actuator_left_joint" type="fixed">
+        <parent link="base_link"/>
+        <child link="actuator_left"/>
+        <origin xyz="-0.205 -0.0760254 0.285" rpy="0 -${pi/7.5} 0"/>
+        <axis xyz="1 0 0"/>
+    </joint>
+    <link name="actuator_left">
+        <visual>
+            <origin xyz="0 0 0"/>
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